File: quadcopter_board/ATmega128RFA1-DevBoard.brd (EAGLE design)
At the start: 57.1 x 53.3 mm, 75 parts, among them J1 ISP, Q1 CJ2302, Q2 CJ2302, Q3 CJ2302, Q4 CJ2302, U1 ATMEGA128RFA1

Commit message: changed component on motor driver
Parts:
- removed C24, C27, C30, C33: 100uf, Seeed-Capacitor-2016:AVX-B
- removed C29, C32: 1uf, Seeed-Capacitor-2016:C0402
- removed C31, C34: 1uf, Seeed-Capacitor-2016:C0603
- removed D6: 28V-5A, Seeed-Diode-2016:DO-214AA
- removed R14, R16: 10K 1/10W, Seeed-Resistor-2016:R0603
- removed R15: 100R, Seeed-Resistor-2016:R0603
- added C12, C13, C35, C36: 1uF, quadparts_prebuilt:CAPC2012X140_HS
- added D7: 360mV, quadparts_prebuilt:SOD3716X135_HS
- added R2: 10K, quadparts_prebuilt:RESC2012X60_HS
- added R3, R4: 100, quadparts_prebuilt:RESC2012X60_HS
- added U$4, U$5, U$6, U$7: 100uF, quadparts:TAJB_SMB_POLAR_CAP
- C23, C26: value 1uf -> 1uF; device Seeed-Capacitor-2016:C0402 -> quadparts_prebuilt:CAPC2012X140_HS
- C25, C28: value 1uf -> 1uF; device Seeed-Capacitor-2016:C0603 -> quadparts_prebuilt:CAPC2012X140_HS
- D3, D4, D5: value 28V-5A -> 360mV; device Seeed-Diode-2016:DO-214AA -> quadparts_prebuilt:SOD3716X135_HS
- R10: value 10K 1/10W -> 100; device Seeed-Resistor-2016:R0603 -> quadparts_prebuilt:RESC2012X60_HS
- R11, R13: value 100R -> 10K; device Seeed-Resistor-2016:R0603 -> quadparts_prebuilt:RESC2012X60_HS
- R12: value 10K 1/10W -> 10K; device Seeed-Resistor-2016:R0603 -> quadparts_prebuilt:RESC2012X60_HS
- R9: value 100R -> 100; device Seeed-Resistor-2016:R0603 -> quadparts_prebuilt:RESC2012X60_HS
- moved D3 186.6 mm to (-14.7, -316.7)
- moved D4 166.4 mm to (-14.7, -319.8)
- moved D5 147.3 mm to (-14.7, -322.8)
- moved R10 141.6 mm to (-16.0, -280.2)
- moved R9 134.7 mm to (-16.0, -277.4)
- moved C23 128.8 mm to (-16.0, -271.8)
- moved R12 122.2 mm to (-16.0, -283.0)
- moved C25 112.0 mm to (-16.0, -260.6)
- moved R11 104.3 mm to (-16.0, -269.0)
- moved C28 103.9 mm to (-16.0, -274.6)
- moved R13 98.9 mm to (-16.0, -285.8)
- moved C26 98.7 mm to (-16.0, -263.4)
Connections:
- net BAT_GND: now also C23.2, C25.2, C26.2, C28.2, R11.1, R13.1, R2.1, U$4.P$2, U$5.P$2, U$6.P$2, U$7.P$2; no longer C23.1, C24.-, C26.1, C27.-, C29.1, C30.-, C32.1, C33.-, R10.1, R14.1, R16.1
- net N$18: now also R12.2; no longer R10.2
- net N$19: now also C12.2, D4.A; no longer C25.1, D3.+
- net N$21: now also R2.2, R3.2; no longer R11.2, R12.2
- net N$22: now also C36.2, D7.A; no longer C28.1, D4.+
- net N$24: now also R10.2; no longer R14.2
- net N$25: now also C13.2, D5.A; no longer C31.1, D5.+
- net N$27: now also R11.2, R4.2; no longer R15.2, R16.2
- net N$28: now also C35.2, D3.A; no longer C34.1, D6.+
- net PB5: now also C23.1; no longer C23.2
- net PE3: now also C28.1, R10.1; no longer C29.2, R13.1
- net PE4: now also C26.1, R4.1; no longer C32.2, R15.1
- net PE5: now also C25.1, R3.1; no longer C26.2, R11.1
- net VCC: now also C12.1, C13.1, C35.1, C36.1, D3.C, D4.C, D5.C, D7.C, U$4.P$1, U$5.P$1, U$6.P$1, U$7.P$1; no longer C24.+, C25.2, C27.+, C28.2, C30.+, C31.2, C33.+, C34.2, D3.-, D4.-, D5.-, D6.-
