File: quadcopter_board/quadcopter.brd (EAGLE design)
At the start: 100 x 80 mm, 75 parts, among them J2 AVR_SPI_PRG_6NS, SW1 PUSHBUTTON_SMD-VERTICAL-1, U2 ATMEGA128RFA1

Commit message: parts placed
Parts:
- moved PIN_3 174.1 mm to (31.0, 31.0), turned to 315 degrees
- moved R16 163.7 mm to (-13.6, 5.30), turned to 270 degrees
- moved R15 161.6 mm to (-11.5, 5.30), turned to 270 degrees
- moved R14 156.3 mm to (-9.30, 5.30), turned to 270 degrees
- moved PIN_8 153.1 mm to (-31.0, 31.0), turned to 225 degrees
- moved D1 148.8 mm to (36.2, -18.0)
- moved R8 146.9 mm to (36.3, -16.1)
- moved C26 144.5 mm to (29.6, -15.2)
- moved D3 143.1 mm to (28.0, -27.6), turned to 45 degrees
- moved PIN_4 141.7 mm to (31.0, -31.0), turned to 45 degrees
- moved SW1 141.0 mm to (-21.2, 3.91), turned to 90 degrees
- moved U$13 138.9 mm to (35.4, 3.56)
- moved C15 134.0 mm to (16.6, -10.6)
- moved C28 132.8 mm to (29.6, 15.2)
- moved B2 132.4 mm to (25.9, 2.75), turned to 180 degrees
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Routing:
- net VCC: track 0.00 -> 81.4 mm
- net 3.3V: track 0.00 -> 20.7 mm
- net BAT_GND: track 0.00 -> 13.0 mm
- net N$25: track 0.00 -> 12.6 mm
- net N$28: track 0.00 -> 12.6 mm
- net N$22: track 0.00 -> 12.6 mm
- net N$19: track 0.00 -> 12.6 mm
- net N$4: track 0.00 -> 11.0 mm
- net N$3: track 0.00 -> 9.80 mm
- net N$17: track 0.00 -> 8.47 mm
- net RFANT: track 0.00 -> 7.47 mm
- net AVDD: track 0.00 -> 5.91 mm
- net N$27: track 0.00 -> 5.87 mm
- net N$18: track 0.00 -> 5.87 mm
- net N$16: track 0.00 -> 5.74 mm
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Other:
- board size 100 x 80 mm -> 115.2 x 115.3 mm
