File: quadcopter-board/quadcopter.brd (EAGLE design)
At the start: 115.2 x 115.3 mm, 75 parts, among them J2 AVR_SPI_PRG_6NS, SW1 PUSHBUTTON_SMD-VERTICAL-1, U2 ATMEGA128RFA1

Commit message: For Design Review
Parts:
- added U$14: (no value), Lab2:UCSD_LOGO
- moved J3 55.2 mm to (11.3, 16.2), turned to 180 degrees
- moved FTDI 33.5 mm to (-36.6, 15.2), turned to 270 degrees
- moved FTDI_(SERIAL_ONLY) 20.4 mm to (-36.6, -2.70), turned to 270 degrees
- moved R16 10.5 mm to (-24.1, 5.30)
- moved U$8 10.5 mm to (-22.0, 0.00)
- moved R14 10.5 mm to (-19.8, 5.30)
- moved R15 10.5 mm to (-22.0, 5.30)
- moved SW1 9.34 mm to (-12.2, 6.41)
- moved C9 8.63 mm to (-12.9, -1.20), turned to 180 degrees
- moved R5 3.04 mm to (5.25, 9.20)
- moved C3 3.04 mm to (0.90, 9.20)
- moved R10 2.00 mm to (26.2, 14.3)
- moved R3 2.00 mm to (-26.2, -14.3)
- moved R4 2.00 mm to (26.2, -14.3)
- moved R9 2.00 mm to (-26.2, 14.3)
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Connections:
- net 3.3V: now also J3.2
- net GND: now also J3.1
- net PB4: now also J3.9; no longer R14.1
- net PB5: now also J3.6
- net PE2: now also R14.1
- net PE3: now also J3.3
- net PE4: now also J3.4
- net PE5: now also J3.5
- net PE6: now also R15.1
- net PE7: now also R16.1
- net PG5: now also J3.10; no longer R15.1
- net SCL: now also J3.8
- net SDA: now also J3.7
Routing:
- net GND: track 0.00 -> 190.9 mm, vias 0 -> 45
- net TX0: track 0.00 -> 86.8 mm, vias 0 -> 1
- net PE5: track 2.56 -> 74.0 mm, vias 0 -> 2
- net RESET: track 0.00 -> 61.9 mm, vias 0 -> 2
- net RX0: track 0.00 -> 61.5 mm, vias 0 -> 1
- net PE6: track 0.00 -> 60.1 mm
- net RX1: track 0.00 -> 60.0 mm, vias 0 -> 2
- net TX1: track 0.00 -> 59.3 mm
- net PE3: track 2.57 -> 59.1 mm, vias 0 -> 1
- net SCL: track 0.00 -> 51.0 mm, vias 0 -> 1
- net PB5: track 2.56 -> 50.0 mm, vias 0 -> 1
- net SDA: track 0.00 -> 45.7 mm, vias 0 -> 2
- net PE4: track 2.56 -> 45.9 mm, vias 0 -> 2
- net PE7: track 0.00 -> 43.2 mm, vias 0 -> 2
- net DTR: track 0.00 -> 39.1 mm
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- added copper zone on layer 15, net 3.3V
- added copper zone on layer 2, net BAT_GND
- added copper zone on layer 1, net GND
- added copper zone on layer 2, net GND
- added copper zone on layer 2, net N$10
- added copper zone on layer 15, net N$11
- added copper zone on layer 2, net N$20
- added copper zone on layer 15, net N$23
- added copper zone on layer 15, net VCC
Other:
- board size 115.2 x 115.3 mm -> 113 x 113 mm
