File: quadcopter-board/quadcopter.brd (EAGLE design)
At the start: 113 x 113 mm, 77 parts, among them J2 AVR_SPI_PRG_6NS, SW1 PUSHBUTTON_SMD-VERTICAL-1, U2 ATMEGA128RFA1

Commit message: Tape-Out
Parts:
- moved C8 48.6 mm to (24.4, -4.45)
- moved C7 48.6 mm to (24.4, -8.88)
Routing:
- net GND: track 191.7 -> 198.1 mm, vias 45 -> 44
- net 3.3V: track 57.1 -> 59.9 mm
- net MISO: track 34.9 -> 36.3 mm
