File: quadcopter-board/quadcopter.sch (EAGLE design)
At the start: 75 parts, among them J2 AVR_SPI_PRG_6NS, SW1 PUSHBUTTON_SMD-VERTICAL-1, U2 ATMEGA128RFA1

Commit message: For Design Review
Connections:
- net 3.3V: now also J3.2
- net GND: now also J3.1
- net PB4: now also J3.9; no longer R14.1
- net PB5: now also J3.6
- net PE2: now also R14.1
- net PE3: now also J3.3
- net PE4: now also J3.4
- net PE5: now also J3.5
- net PE6: now also R15.1
- net PE7: now also R16.1
- net PG5: now also J3.10; no longer R15.1
- net SCL: now also J3.8
- net SDA: now also J3.7
Changed lines of the file:
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@@
 <layers>
 <layer number="1" name="Top" color="4" fill="1" visible="no" active="no"/>
+<layer number="2" name="Route2" color="1" fill="3" visible="no" active="no"/>
+<layer number="3" name="Route3" color="4" fill="3" visible="no" active="no"/>
+<layer number="4" name="Route4" color="1" fill="4" visible="no" active="no"/>
+<layer number="5" name="Route5" color="4" fill="4" visible="no" active="no"/>
+<layer number="6" name="Route6" color="1" fill="8" visible="no" active="no"/>
+<layer number="7" name="Route7" color="4" fill="8" visible="no" active="no"/>
+<layer number="8" name="Route8" color="1" fill="2" visible="no" active="no"/>
+<layer number="9" name="Route9" color="4" fill="2" visible="no" active="no"/>
+<layer number="10" name="Route10" color="1" fill="7" visible="no" active="no"/>
+<layer number="11" name="Route11" color="4" fill="7" visible="no" active="no"/>
+<layer number="13" name="Route13" color="4" fill="5" visible="no" active="no"/>
+<layer number="14" name="Route14" color="1" fill="6" visible="no" active="no"/>
+<layer number="15" name="Route15" color="4" fill="6" visible="no" active="no"/>
 <layer number="16" name="Bottom" color="1" fill="1" visible="no" active="no"/>
 <layer number="17" name="Pads" color="2" fill="1" visible="no" active="no"/>
@@
 <part name="GND27" library="SparkFun-Aesthetics" deviceset="GND" device=""/>
 <part name="GND9" library="SparkFun-Aesthetics" deviceset="GND" device=""/>
-<part name="U$3" library="quadparts" deviceset="RESISTOR" device="" value="0"/>
 <part name="GND24" library="SparkFun-Aesthetics" deviceset="GND" device=""/>
 <part name="GND32" library="SparkFun-Aesthetics" deviceset="GND" device=""/>
@@
 <part name="GND15" library="SparkFun" deviceset="GND" device=""/>
 <part name="GND16" library="SparkFun" deviceset="GND" device=""/>
+<part name="GND17" library="SparkFun" deviceset="GND" device=""/>
+<part name="P+1" library="SparkFun-Aesthetics" deviceset="3.3V" device=""/>
+<part name="U$3" library="quadparts" deviceset="RESISTOR" device="" value="0"/>
 </parts>
 <sheets>
@@
 <instance part="GND27" gate="1" x="297.18" y="36.83"/>
 <instance part="GND9" gate="1" x="246.38" y="46.99"/>
-<instance part="U$3" gate="G$1" x="190.5" y="34.29"/>
 <instance part="GND24" gate="1" x="208.28" y="26.67"/>
 <instance part="GND32" gate="1" x="293.37" y="215.9"/>
@@
 <instance part="GND15" gate="1" x="299.72" y="128.27"/>
 <instance part="GND16" gate="1" x="240.03" y="171.45"/>
+<instance part="GND17" gate="1" x="372.11" y="125.73"/>
+<instance part="P+1" gate="G$1" x="410.21" y="133.35"/>
+<instance part="U$3" gate="G$1" x="190.5" y="34.29"/>
 </instances>
 <busses>
@@
 </segment>
 <segment>
-<pinref part="U$3" gate="G$1" pin="P$2"/>
 <pinref part="GND24" gate="1" pin="GND"/>
 <wire x1="198.12" y1="34.29" x2="208.28" y2="34.29" width="0.1524" layer="91"/>
 <wire x1="208.28" y1="34.29" x2="208.28" y2="29.21" width="0.1524" layer="91"/>
+<pinref part="U$3" gate="G$1" pin="P$2"/>
 </segment>
 <segment>
@@
 <wire x1="240.03" y1="185.42" x2="240.03" y2="173.99" width="0.1524" layer="91"/>
 </segment>
+<segment>
+<pinref part="J3" gate="G$1" pin="1"/>
+<pinref part="GND17" gate="1" pin="GND"/>
+<wire x1="372.11" y1="128.27" x2="368.3" y2="128.27" width="0.1524" layer="91"/>
+</segment>
 </net>
 <net name="N$3" class="0">
@@
 </segment>
 <segment>
-<pinref part="R15" gate="G$1" pin="1"/>
-<wire x1="256.54" y1="147.32" x2="250.19" y2="147.32" width="0.1524" layer="91"/>
+<pinref part="J3" gate="G$1" pin="10"/>
+<wire x1="368.3" y1="151.13" x2="377.19" y2="151.13" width="0.1524" layer="91"/>
 </segment>
 </net>
@@
 <pinref part="U2" gate="G$1" pin="PE7(ICP3/INT7/CLKO)"/>
 </segment>
+<segment>
+<pinref part="R16" gate="G$1" pin="1"/>
+<wire x1="256.54" y1="137.16" x2="251.46" y2="137.16" width="0.1524" layer="91"/>
+</segment>
 </net>
 <net name="PE6" class="0">
@@
 <label x="24.13" y="175.26" size="1.27" layer="95" rot="MR0" xref="yes"/>
 <pinref part="U2" gate="G$1" pin="PE6(T3/INT6)"/>
+</segment>
+<segment>
+<pinref part="R15" gate="G$1" pin="1"/>
+<wire x1="256.54" y1="147.32" x2="250.19" y2="147.32" width="0.1524" layer="91"/>
 </segment>
 </net>
@@
 <pinref part="C25" gate="G$1" pin="1"/>
 </segment>
+<segment>
+<pinref part="J3" gate="G$1" pin="5"/>
+<wire x1="368.3" y1="138.43" x2="378.46" y2="138.43" width="0.1524" layer="91"/>
+</segment>
 </net>
 <net name="PE4" class="0">
@@
 <junction x="21.59" y="30.48"/>
 </segment>
+<segment>
+<pinref part="J3" gate="G$1" pin="4"/>
+<wire x1="368.3" y1="135.89" x2="378.46" y2="135.89" width="0.1524" layer="91"/>
+</segment>
 </net>
 <net name="PE3" class="0">
@@
 <junction x="21.59" y="91.44"/>
 </segment>
+<segment>
+<pinref part="J3" gate="G$1" pin="3"/>
+<wire x1="368.3" y1="133.35" x2="378.46" y2="133.35" width="0.1524" layer="91"/>
+</segment>
 </net>
 <net name="PE2" class="0">
@@
 <label x="24.13" y="185.42" size="1.27" layer="95" rot="MR0" xref="yes"/>
 <pinref part="U2" gate="G$1" pin="PE2(XCK0/AIN0)"/>
+</segment>
+<segment>
+<pinref part="R14" gate="G$1" pin="1"/>
+<wire x1="256.54" y1="157.48" x2="250.19" y2="157.48" width="0.1524" layer="91"/>
 </segment>
 </net>
@@
 <label x="381" y="24.13" size="1.778" layer="95" rot="R180" xref="yes"/>
 </segment>
+<segment>
+<pinref part="J3" gate="G$1" pin="7"/>
+<wire x1="368.3" y1="143.51" x2="377.19" y2="143.51" width="0.1524" layer="91"/>
+</segment>
 </net>
 <net name="SCL" class="0">
@@
 <wire x1="381" y1="31.75" x2="384.81" y2="31.75" width="0.1524" layer="91"/>
 <label x="381" y="31.75" size="1.778" layer="95" rot="R180" xref="yes"/>
+</segment>
+<segment>
+<pinref part="J3" gate="G$1" pin="8"/>
+<wire x1="368.3" y1="146.05" x2="377.19" y2="146.05" width="0.1524" layer="91"/>
 </segment>
 </net>
@@
 <junction x="86.36" y="91.44"/>
 </segment>
+<segment>
+<pinref part="J3" gate="G$1" pin="6"/>
+<wire x1="368.3" y1="140.97" x2="378.46" y2="140.97" width="0.1524" layer="91"/>
+</segment>
 </net>
 <net name="PB4" class="0">
@@
 </segment>
 <segment>
-<pinref part="R14" gate="G$1" pin="1"/>
-<wire x1="256.54" y1="157.48" x2="250.19" y2="157.48" width="0.1524" layer="91"/>
+<pinref part="J3" gate="G$1" pin="9"/>
+<wire x1="368.3" y1="148.59" x2="377.19" y2="148.59" width="0.1524" layer="91"/>
 </segment>
 </net>
@@
 <junction x="337.82" y="44.45"/>
 </segment>
+<segment>
+<pinref part="J3" gate="G$1" pin="2"/>
+<pinref part="P+1" gate="G$1" pin="3.3V"/>
+<wire x1="368.3" y1="130.81" x2="410.21" y2="130.81" width="0.1524" layer="91"/>
+<wire x1="410.21" y1="130.81" x2="410.21" y2="133.35" width="0.1524" layer="91"/>
+</segment>
 </net>
 <net name="VCC" class="0">
@@
 <pinref part="GND33" gate="1" pin="BAT_GND"/>
 <wire x1="177.8" y1="39.37" x2="177.8" y2="34.29" width="0.1524" layer="91"/>
-<pinref part="U$3" gate="G$1" pin="P$1"/>
 <wire x1="177.8" y1="34.29" x2="177.8" y2="31.75" width="0.1524" layer="91"/>
 <wire x1="187.96" y1="34.29" x2="177.8" y2="34.29" width="0.1524" layer="91"/>
 <junction x="177.8" y="34.29"/>
-</segment>
-<segment>
+<pinref part="U$3" gate="G$1" pin="P$1"/>
+</segment>
+<segment>
